File: board/board.kicad_pcb (KiCad board)
At the start: 2 copper layers, 21 x 13 mm, 1 part

Commit message: initial
Parts:
- removed LOGO1: Logo_Open_Hardware_Small, Symbol:OSHW-Symbol_6.7x6mm_SilkScreen
- added J1: Conn_01x10_Male, on_edge:on_edge_2x05_host, F.Cu at (67.5, 133.0)
- added J2: Conn_01x10_Male, on_edge:on_edge_2x05_solder, F.Cu at (67.5, 140.0)
Routing:
- net Net-(J1-Pad8): track 0.00 -> 4.90 mm
- net Net-(J1-Pad7): track 0.00 -> 4.90 mm
- net Net-(J1-Pad5): track 0.00 -> 4.65 mm
- net Net-(J1-Pad4): track 0.00 -> 4.65 mm
- net Net-(J1-Pad1): track 0.00 -> 4.65 mm
- net Net-(J1-Pad9): track 0.00 -> 4.60 mm
- net Net-(J1-Pad6): track 0.00 -> 4.60 mm
- net Net-(J1-Pad10): track 0.00 -> 4.50 mm
- net Net-(J1-Pad3): track 0.00 -> 3.40 mm
- net Net-(J1-Pad2): track 0.00 -> 3.40 mm
Other:
- board size 21 x 13 mm -> 10 x 9 mm
- rule pad_to_mask_clearance: 0 -> 0.04
