File: board/board.kicad_sch (KiCad schematic)
At the start: 1 part

Commit message: initial
Parts:
- removed LOGO1: Logo_Open_Hardware_Small, Symbol:OSHW-Symbol_6.7x6mm_SilkScreen, symbol Graphic:Logo_Open_Hardware_Small
- added J1: Conn_01x10_Male, on_edge:on_edge_2x05_host, symbol Connector:Conn_01x10_Male
- added J2: Conn_01x10_Male, on_edge:on_edge_2x05_solder, symbol Connector:Conn_01x10_Male
Connections:
- new net: J1.1 (Pin_1), J2.1 (Pin_1)
- new net: J1.10 (Pin_10), J2.10 (Pin_10)
- new net: J1.2 (Pin_2), J2.2 (Pin_2)
- new net: J1.3 (Pin_3), J2.3 (Pin_3)
- new net: J1.4 (Pin_4), J2.4 (Pin_4)
- new net: J1.5 (Pin_5), J2.5 (Pin_5)
- new net: J1.6 (Pin_6), J2.6 (Pin_6)
- new net: J1.7 (Pin_7), J2.7 (Pin_7)
- new net: J1.8 (Pin_8), J2.8 (Pin_8)
- new net: J1.9 (Pin_9), J2.9 (Pin_9)
Other:
- removed sheet implementation
- note removed: "Input connectors go here"
- note removed: "Output connectors go here"
Changed lines of the file:
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@@
 (kicad_sch (version 20211123) (generator eeschema)
   (paper "A4")
-  (text "Output connectors go here" (at 224.79 88.9 0)
-    (effects (font (size 1.27 1.27)) (justify left bottom))
+  (wire (pts (xy 99.06 99.06) (xy 92.075 99.06))
+    (stroke (width 0) (type default) (color 0 0 0 0))
   )
-  (text "Input connectors go here" (at 49.53 88.9 0)
-    (effects (font (size 1.27 1.27)) (justify left bottom))
+  (wire (pts (xy 99.06 109.22) (xy 92.075 109.22))
+    (stroke (width 0) (type default) (color 0 0 0 0))
   )
-  (symbol (lib_id "Graphic:Logo_Open_Hardware_Small") (at 273.05 157.48 0) (unit 1)
-    (in_bom yes) (on_board yes) (fields_autoplaced)
-    (property "Reference" "LOGO1" (id 0) (at 273.05 150.495 0)
+  (wire (pts (xy 92.075 106.68) (xy 99.06 106.68))
+    (stroke (width 0) (type default) (color 0 0 0 0))
+  )
+  (wire (pts (xy 92.075 111.76) (xy 99.06 111.76))
+    (stroke (width 0) (type default) (color 0 0 0 0))
+  )
+  (wire (pts (xy 92.075 96.52) (xy 99.06 96.52))
+    (stroke (width 0) (type default) (color 0 0 0 0))
+  )
+  (wire (pts (xy 99.06 114.3) (xy 92.075 114.3))
+    (stroke (width 0) (type default) (color 0 0 0 0))
+  )
+  (wire (pts (xy 92.075 91.44) (xy 99.06 91.44))
+    (stroke (width 0) (type default) (color 0 0 0 0))
+  )
+  (wire (pts (xy 99.06 104.14) (xy 92.075 104.14))
+    (stroke (width 0) (type default) (color 0 0 0 0))
+  )
+  (wire (pts (xy 92.075 101.6) (xy 99.06 101.6))
+    (stroke (width 0) (type default) (color 0 0 0 0))
+  )
+  (wire (pts (xy 99.06 93.98) (xy 92.075 93.98))
+    (stroke (width 0) (type default) (color 0 0 0 0))
+  )
+  (symbol (lib_id "Connector:Conn_01x10_Male") (at 86.995 101.6 0)
+    (in_bom yes) (on_board yes)
+    (property "Reference" "J1" (id 0) (at 89.7382 86.8426 0))
+    (property "Value" "Conn_01x10_Male" (id 1) (at 89.7382 89.154 0))
+    (property "Footprint" "on_edge:on_edge_2x05_host" (id 2) (at 86.995 101.6 0)
       (effects (font (size 1.27 1.27)) hide)
     )
-    (property "Value" "Logo_Open_Hardware_Small" (id 1) (at 273.05 163.195 0)
+    (property "Datasheet" "~" (id 3) (at 86.995 101.6 0)
       (effects (font (size 1.27 1.27)) hide)
     )
-    (property "Footprint" "Symbol:OSHW-Symbol_6.7x6mm_SilkScreen" (id 2) (at 273.05 157.48 0)
+    (pin "1")
+    (pin "10")
+    (pin "2")
+    (pin "3")
+    (pin "4")
+    (pin "5")
+    (pin "6")
+    (pin "7")
+    (pin "8")
+    (pin "9")
+  )
+  (symbol (lib_id "Connector:Conn_01x10_Male") (at 93.98 101.6 0)
+    (in_bom yes) (on_board yes)
+    (property "Reference" "J2" (id 0) (at 96.7232 86.8426 0))
+    (property "Value" "Conn_01x10_Male" (id 1) (at 96.7232 89.154 0))
+    (property "Footprint" "on_edge:on_edge_2x05_solder" (id 2) (at 93.98 101.6 0)
       (effects (font (size 1.27 1.27)) hide)
     )
-    (property "Datasheet" "~" (id 3) (at 273.05 157.48 0)
+    (property "Datasheet" "~" (id 3) (at 93.98 101.6 0)
       (effects (font (size 1.27 1.27)) hide)
     )
-  )
-  (sheet (at 114.3 72.39) (size 60.96 62.23) (fields_autoplaced)
-    (stroke (width 0.1524) (type solid) (color 0 0 0 0))
-    (fill (color 0 0 0 0.0000))
-    (property "Sheet name" "implementation" (id 0) (at 114.3 71.6784 0)
-      (effects (font (size 1.27 1.27)) (justify left bottom))
-    )
-    (property "Sheet file" "implementation.kicad_sch" (id 1) (at 114.3 135.2046 0)
-      (effects (font (size 1.27 1.27)) (justify left top))
-    )
+    (pin "1")
+    (pin "10")
+    (pin "2")
+    (pin "3")
+    (pin "4")
+    (pin "5")
+    (pin "6")
+    (pin "7")
+    (pin "8")
+    (pin "9")
   )
   (sheet_instances
     (path "/" (page "1"))
-    (path "/767ce4c6-0e55-4543-92f0-34cb8237a544" (page "2"))
   )
   (symbol_instances
-    (path "/b72b6f4a-7489-40f2-bb90-d75ae01aa368"
-      (reference "LOGO1") (unit 1) (value "Logo_Open_Hardware_Small") (footprint "Symbol:OSHW-Symbol_6.7x6mm_SilkScreen")
+    (path "/00000000-0000-0000-0000-0000602c6b82"
+      (reference "J1") (unit 1) (value "Conn_01x10_Male") (footprint "on_edge:on_edge_2x05_host")
+    )
+    (path "/00000000-0000-0000-0000-0000602c6b88"
+      (reference "J2") (unit 1) (value "Conn_01x10_Male") (footprint "on_edge:on_edge_2x05_solder")
     )
   )
